File: Schematic/VGA_and_ADC.kicad_sch (KiCad schematic)
At the start: 20 parts, among them J4 HDMI_A breakout, J5 VGA in, U10 ADC1175-50CIMTX/NOPB, U11 ADC1175-50CIMTX/NOPB, U12 ADC1175-50CIMTX/NOPB

Commit message: updated make and circuit
Parts:
- removed C_bypassBA, C_bypassBD, C_bypassGA, C_bypassGD: 0.1uF, symbol Device:C_Small
- removed FB1, FB3: FerriteBead, symbol Device:FerriteBead
- removed U11, U12: ADC1175-50CIMTX/NOPB, PW24_TEX, symbol ADC:ADC1175-50CIMTX_NOPB
- added R13: 2.7k, symbol Device:R_US
- added R8: 1k, symbol Device:R_US
- added R9: 470, symbol Device:R_US
- renumbered C_bypassRA to C_bypassA, C_bypassRD to C_bypassD, J4 to J9
Connections:
- net Analog VDD: now also C_bypassD.2, U10.11 (DVDD), U10.13 (DVDD)
- net GND: now also C_bypassA.1, C_decouple1.1, J5.6, J5.7, J5.8, R10.1, R11.1, R12.1, R5.1, R7.1, U10.24 (DVSS); no longer U10.11 (DVDD)
- net VGA_B: now also R13.1
- net VGA_G: now also R9.1
- net VGA_R: now also R8.1; no longer U10.19 (VIN)
- net 8051 C0: now reaches U10.5 (D2)
- net 8051 C1: now reaches U10.6 (D3)
- net 8051 C2: now reaches U10.7 (D4)
- net 8051 R0 renamed 8051 C3
- net 8051 R1 renamed 8051 C4
- removed net Analog GND: C_bypassA.1, C_decouple1.1, J5.6, J5.7, J5.8, R10.1, R11.1, R12.1, R5.1, R7.1, U10.20 (AVSS), U10.21 (AVSS)
- removed net MAIN_VCC: C_bypassD.2, U10.13 (DVDD), U10.24 (DVSS)
- new net: R13.2, R8.2, R9.2, U10.19 (VIN)
- new net VGA_GND: U10.20 (AVSS), U10.21 (AVSS)
Other:
- moved on the sheet: C_bypassA, C_bypassD, C_decouple1, R10, R11, R12, R4, R5, R7

Commit message: final hardware schematic
Parts:
- added U9: SN74AHCT14-W, PW14_TEX, symbol 2026-04-29_06-18-06:SN74AHCT14-W
Connections:
- net ALE: now also U9.11 (5A); no longer U10.12 (CLK)
- net Analog VDD: now also U9.14 (VCC)
- net GND: now also U9.1 (1A), U9.13 (6A), U9.3 (2A), U9.5 (3A), U9.7 (GND)
- new net: U9.10 (5Y), U9.9 (4A)
- new net CLK: U10.12 (CLK), U9.8 (4Y)
